File: hardware/alpha_board_05a.sch (EAGLE design)
At the start: 18 parts

Commit message: few bug changes
Parts:
- removed R6: 0, SparkFun:RESISTOR1206
Connections:
- removed net GNDR: DHT03_EXT.3, DHT03_INT.3, R6.1
- net GND: now also DHT03_EXT.3, DHT03_INT.3; no longer R6.2
Changed lines of the file:
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@@
 <?xml version="1.0" encoding="utf-8"?>
 <!DOCTYPE eagle SYSTEM "eagle.dtd">
-<eagle version="7.4.0">
+<eagle version="6.6.0">
 <drawing>
 <settings>
@@
 <part name="DHT03_EXT" library="SparkFun" deviceset="M03" device="LOCK"/>
 <part name="ADC" library="SparkFun-Connectors" deviceset="M04" device="LOCK_LONGPADS"/>
-<part name="R6" library="SparkFun" deviceset="RESISTOR" device="1206" value="0"/>
 <part name="AUDIO" library="SparkFun" deviceset="M03" device="LOCK"/>
 <part name="U$2" library="calculator_lib" deviceset="MICROSD-HIROSE" device=""/>
@@
 <part name="D1" library="diode" deviceset="DIODE-" device="SOD323-W"/>
 <part name="G1" library="Simplex-Battery" deviceset="HU2032-LF" device=""/>
+<part name="GND1" library="supply1" deviceset="GND" device=""/>
 </parts>
 <sheets>
@@
 <instance part="DHT03_EXT" gate="G$1" x="121.92" y="35.56" rot="R180"/>
 <instance part="ADC" gate="G$1" x="58.42" y="-30.48" rot="R90"/>
-<instance part="R6" gate="G$1" x="93.98" y="33.02" rot="R180"/>
 <instance part="AUDIO" gate="G$1" x="-30.48" y="2.54"/>
 <instance part="U$2" gate="G$1" x="-48.26" y="17.78" rot="R180"/>
@@
 <instance part="D1" gate="G$1" x="38.1" y="63.5" rot="R180"/>
 <instance part="G1" gate="BAT" x="48.26" y="63.5" rot="R180"/>
+<instance part="GND1" gate="1" x="101.6" y="10.16"/>
 </instances>
 <busses>
@@
 </segment>
 <segment>
-<pinref part="R6" gate="G$1" pin="2"/>
 <wire x1="88.9" y1="33.02" x2="88.9" y2="30.48" width="0.1524" layer="91"/>
 <pinref part="GND2" gate="1" pin="GND"/>
+<pinref part="DHT03_EXT" gate="G$1" pin="3"/>
+<wire x1="114.3" y1="33.02" x2="88.9" y2="33.02" width="0.1524" layer="91"/>
+<label x="101.6" y="33.02" size="1.778" layer="95"/>
 </segment>
 <segment>
@@
 <wire x1="114.3" y1="-22.86" x2="101.6" y2="-22.86" width="0.1524" layer="91"/>
 <label x="101.6" y="-27.94" size="1.778" layer="95"/>
+<label x="104.14" y="-22.86" size="1.778" layer="95"/>
 </segment>
 <segment>
@@
 <pinref part="G1" gate="BAT" pin="-"/>
 <wire x1="53.34" y1="63.5" x2="63.5" y2="63.5" width="0.1524" layer="91"/>
+</segment>
+<segment>
+<pinref part="DHT03_INT" gate="G$1" pin="3"/>
+<wire x1="114.3" y1="12.7" x2="101.6" y2="12.7" width="0.1524" layer="91"/>
+<pinref part="GND1" gate="1" pin="GND"/>
 </segment>
 </net>
@@
 </segment>
 </net>
-<net name="GNDR" class="0">
-<segment>
-<pinref part="DHT03_EXT" gate="G$1" pin="3"/>
-<wire x1="114.3" y1="33.02" x2="99.06" y2="33.02" width="0.1524" layer="91"/>
-<pinref part="R6" gate="G$1" pin="1"/>
-<label x="101.6" y="33.02" size="1.778" layer="95"/>
-</segment>
-<segment>
-<pinref part="DHT03_INT" gate="G$1" pin="3"/>
-<wire x1="114.3" y1="12.7" x2="93.98" y2="12.7" width="0.1524" layer="91"/>
-<label x="101.6" y="12.7" size="1.778" layer="95"/>
-</segment>
-</net>
